File: Power/Power.kicad_sch (KiCad schematic)
At the start: 62 parts, among them J1 Conn_01x01, J2 Conn_01x04, Q1 AOD417, Q2 2N7002, Q3 AOD417, Q4 HSU60P02, SW1 SW_SPDT, U1 CN3765, U2 FP6188XR-G1, U3 FP6296XR-G1

Commit message: update
Parts:
- added C13: 22u, Capacitor_SMD:C_0805_2012Metric, symbol 0805:C
- renumbered C13 to C14, C14 to C15, C15 to C16, C16 to C17, C17 to C18, C18 to C19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
Connections:
- net GND: now also DC1.5, DC2.5, C13.2
- net at C14.1, C15.1, C16.1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: now also C13.1
Other:
- moved on the sheet: C14, C15
