File: Power/Power.kicad_pcb (KiCad board)
At the start: 2 copper layers, 90 x 25 mm, 62 parts, among them J1 Conn_01x01, J2 Conn_01x04, Q1 AOD417, Q2 2N7002, Q3 AOD417, Q4 HSU60P02, SW1 SW_SPDT, U1 CN3765, U2 FP6188XR-G1, U3 FP6296XR-G1

Commit message: update
Parts:
- added C13: 22u, Capacitor_SMD:C_0805_2012Metric, F.Cu at (236.9, 116.6)
- moved BT1 125.7 mm to (218.6, 125.7), turned to -90 degrees
- moved U1 122.2 mm to (190.0, 122.1), turned to 90 degrees
- moved L1 108.7 mm to (205.0, 128.0)
- moved Q3 106.6 mm to (187.9, 128.3), turned to 180 degrees
- moved C23 99.4 mm to (221.4, 122.1)
- moved C2 99.1 mm to (183.5, 119.8), turned to 180 degrees
- moved C21 98.7 mm to (221.8, 117.6)
- moved C22 96.8 mm to (221.4, 120.0)
- moved Q4 94.1 mm to (239.8, 125.8), turned to -90 degrees
- moved C1 90.9 mm to (183.5, 121.9), turned to 180 degrees
- moved R7 76.4 mm to (242.1, 113.1)
- moved C3 75.9 mm to (183.5, 124.0), turned to 180 degrees
- moved L3 75.8 mm to (234.8, 111.3), turned to 180 degrees
- moved U3 74.9 mm to (231.1, 119.6), turned to -90 degrees
- moved R3 73.6 mm to (205.6, 112.6), turned to -90 degrees
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- renumbered C13 to C14, C14 to C15, C15 to C16, C16 to C17, C17 to C18, C18 to C19, C19 to C20, C20 to C21, C21 to C22, C22 to C23
Connections:
- DC1 pad 5: Net-(DC1-Pad5) -> GND
- DC2 pad 5: Net-(DC1-Pad5) -> GND
Routing:
- net Net-(DC1-Pad4): track 0.00 -> 50.3 mm, vias 0 -> 4
- net Net-(R4-Pad2): track 0.00 -> 33.0 mm, vias 0 -> 2
- net Net-(R4-Pad3): track 0.00 -> 30.5 mm, vias 0 -> 2
- net Net-(R5-Pad2): track 0.00 -> 26.3 mm, vias 0 -> 2
- net /EN: track 0.00 -> 23.8 mm, vias 0 -> 2
- net Net-(BT1-Pad1): track 0.00 -> 22.5 mm
- net Net-(D1-Pad1): track 0.00 -> 21.3 mm
- net Net-(D2-Pad1): track 0.00 -> 20.4 mm
- net Net-(C21-Pad1): track 0.00 -> 15.6 mm, vias 0 -> 2
- net Net-(R15-Pad1): track 0.00 -> 13.0 mm, vias 0 -> 2
- net +5V: track 0.00 -> 12.8 mm
- net Net-(D6-Pad2): track 0.00 -> 12.5 mm
- net Net-(D3-Pad1): track 0.00 -> 12.0 mm
- net Net-(C13-Pad1): track 0.00 -> 11.6 mm, vias 0 -> 2
- net Net-(Q4-Pad1): track 0.00 -> 11.6 mm
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- added copper zone on F.Cu, net +12V
- added copper zone on F.Cu, net +5V
- added copper zone on B.Cu, net GND
- added copper zone on F.Cu, net Net-(BT1-Pad1)
- added copper zone on F.Cu, net Net-(C1-Pad1)
- added copper zone on F.Cu, net Net-(C13-Pad1)
- added copper zone on F.Cu, net Net-(C21-Pad1)

Commit message: update
Parts:
- moved C1 63.1 mm to (128.3, 91.2)
- moved C2 63.1 mm to (128.3, 89.2)
- moved C3 63.1 mm to (128.3, 93.3)
- moved C21 63.0 mm to (166.6, 87.2)
- moved C22 63.0 mm to (166.2, 89.6)
- moved C23 63.0 mm to (166.2, 91.7)
- moved D1 63.0 mm to (150.3, 78.6)
- moved DC2 63.0 mm to (156.8, 84.6)
- moved J2 63.0 mm to (120.9, 81.1)
- moved L3 63.0 mm to (179.6, 80.9)
- moved Q1 63.0 mm to (122.8, 95.6)
- moved Q2 63.0 mm to (112.8, 99.4)
- moved Q3 63.0 mm to (132.7, 97.9)
- moved Q4 63.0 mm to (184.6, 95.4)
- moved R11 63.0 mm to (171.7, 87.4)
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Routing:
- net Net-(DC1-Pad4): track 50.3 -> 127.4 mm
- net Net-(BT1-Pad1): track 22.5 -> 36.3 mm, vias 0 -> 2
Other:
- board text added: "+"
- board text added: "-"
