File: Led_Control_Circuit/Led_Control_Circuit.kicad_sch (KiCad schematic)
At the start: 1 part

Commit message: update
Parts:
- added J?: USB_C_Receptacle_USB2.0, Connector_USB:USB_C_Receptacle_HRO_TYPE-C-31-M-12, symbol Connector:USB_C_Receptacle_USB2.0
- added U?: AMS1117-3.3, Package_TO_SOT_SMD:SOT-223-3_TabPin2, symbol Regulator_Linear:AMS1117-3.3
- U?: footprint Espressif:ESP32-S3-WROOM-1 -> Espressif:ESP32-S3-WROOM-1U
Connections:
- new net: J?.A1 (GND), J?.A12 (GND), J?.B1 (GND), J?.B12 (GND)
- new net: J?.A4 (VBUS), J?.A9 (VBUS), J?.B4 (VBUS), J?.B9 (VBUS)
Changed lines of the file:
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@@
     (property "Reference" "U?" (id 0) (at 148.59 25.4 0))
     (property "Value" "ESP32-S3-WROOM-1" (id 1) (at 148.59 27.94 0))
-    (property "Footprint" "Espressif:ESP32-S3-WROOM-1" (id 2) (at 149.225 104.775 0)
+    (property "Footprint" "Espressif:ESP32-S3-WROOM-1U" (id 2) (at 149.225 104.775 0)
       (effects (font (size 1.27 1.27)) hide)
     )
@@
     (pin "9")
   )
+  (symbol (lib_id "Connector:USB_C_Receptacle_USB2.0") (at 36.83 82.55 0) (unit 1)
+    (in_bom yes) (on_board yes) (fields_autoplaced)
+    (property "Reference" "J?" (id 0) (at 36.83 59.69 0))
+    (property "Value" "USB_C_Receptacle_USB2.0" (id 1) (at 36.83 62.23 0))
+    (property "Footprint" "Connector_USB:USB_C_Receptacle_HRO_TYPE-C-31-M-12" (id 2) (at 40.64 82.55 0)
+      (effects (font (size 1.27 1.27)) hide)
+    )
+    (property "Datasheet" "https://www.usb.org/sites/default/files/documents/usb_type-c.zip" (id 3) (at 40.64 82.55 0)
+      (effects (font (size 1.27 1.27)) hide)
+    )
+    (pin "A1")
+    (pin "A12")
+    (pin "A4")
+    (pin "A5")
+    (pin "A6")
+    (pin "A7")
+    (pin "A8")
+    (pin "A9")
+    (pin "B1")
+    (pin "B12")
+    (pin "B4")
+    (pin "B5")
+    (pin "B6")
+    (pin "B7")
+    (pin "B8")
+    (pin "B9")
+    (pin "S1")
+  )
+  (symbol (lib_id "Regulator_Linear:AMS1117-3.3") (at 46.99 133.35 0) (unit 1)
+    (in_bom yes) (on_board yes) (fields_autoplaced)
+    (property "Reference" "U?" (id 0) (at 46.99 125.73 0))
+    (property "Value" "AMS1117-3.3" (id 1) (at 46.99 128.27 0))
+    (property "Footprint" "Package_TO_SOT_SMD:SOT-223-3_TabPin2" (id 2) (at 46.99 128.27 0)
+      (effects (font (size 1.27 1.27)) hide)
+    )
+    (property "Datasheet" "http://www.advanced-monolithic.com/pdf/ds1117.pdf" (id 3) (at 49.53 139.7 0)
+      (effects (font (size 1.27 1.27)) hide)
+    )
+    (pin "1")
+    (pin "2")
+    (pin "3")
+  )
   (sheet_instances
     (path "/" (page "1"))
   )
   (symbol_instances
+    (path "/7ea7cc4a-9f54-4274-8035-370397e0f165"
+      (reference "J?") (unit 1) (value "USB_C_Receptacle_USB2.0") (footprint "Connector_USB:USB_C_Receptacle_HRO_TYPE-C-31-M-12")
+    )
     (path "/47fbb966-03d1-48bd-bed6-43dfb61139c5"
-      (reference "U?") (unit 1) (value "ESP32-S3-WROOM-1") (footprint "Espressif:ESP32-S3-WROOM-1")
+      (reference "U?") (unit 1) (value "ESP32-S3-WROOM-1") (footprint "Espressif:ESP32-S3-WROOM-1U")
+    )
+    (path "/d8a0a197-bf2d-4960-87f8-d261881d2594"
+      (reference "U?") (unit 1) (value "AMS1117-3.3") (footprint "Package_TO_SOT_SMD:SOT-223-3_TabPin2")
     )
   )

Commit message: updater
Parts:
- added C1, C7: 0.1u, Capacitor_SMD:C_0805_2012Metric, symbol 1CommonUse:C0805
- added C2, C3, C5, C6: 1u, Capacitor_SMD:C_0805_2012Metric, symbol 1CommonUse:C0805
- added C4: 10u, Capacitor_SMD:C_0805_2012Metric, symbol 1CommonUse:C0805
- added Card1: TF-01A, SDCard:TF-SMD_TF-01A, symbol SDCard:TF-01A
- added D1, D3: 1N5819HW, Diode_SMD:D_SOD-123, symbol Device:D
- added D2: LED0805, LED_SMD:LED_0805_2012Metric, symbol 1CommonUse:LED0805
- added J2: Conn_01x02, 1Comment:Battery, symbol Connector_Generic:Conn_01x02
- added J3: Conn_01x20, Connector_PinSocket_2.54mm:PinSocket_2x10_P2.54mm_Vertical_SMD, symbol Connector_Generic:Conn_01x20
- added R1: 5.1K, Resistor_SMD:R_0805_2012Metric, symbol 1CommonUse:R0805
- added R2: 1k, Resistor_SMD:R_0805_2012Metric, symbol 1CommonUse:R0805
- added R3: 1K, Resistor_SMD:R_0805_2012Metric, symbol 1CommonUse:R0805
- added R4, R5, R6, R7: 3.3K, Resistor_SMD:R_0805_2012Metric, symbol 1CommonUse:R0805
- added SW1: SW_Push, Button_Switch_SMD:SW_SPST_CK_RS282G05A3, symbol Switch:SW_Push
- added TP1: TestPoint_2Pole, Connector_PinHeader_2.00mm:PinHeader_1x02_P2.00mm_Vertical, symbol Connector:TestPoint_2Pole
- added U1: 74LVC125, Package_SO:TSSOP-14_4.4x5mm_P0.65mm, symbol 74xx:74LVC125
- J1: renamed from J?; footprint Connector_USB:USB_C_Receptacle_HRO_TYPE-C-31-M-12 -> 1Comment:USB_C_Receptacle_HRO_TYPE-C-31-M-12
- gave numbers to parts that had none: 2
Connections:
- net GND: now reaches U3.1 (GND)
- net GND: now also J1.A1 (GND), J1.A12 (GND), J1.B1 (GND), J1.B12 (GND), J1.S1 (SHIELD), U2.1 (GND), U3.40 (GND), U3.41 (GND), C1.2, C2.2, C3.2, C4.2, C5.2, C6.1, C7.2, Card1.10 (GND), Card1.11 (GND), Card1.12 (GND), Card1.13 (GND), Card1.6 (VSS), D2.1 (K), J2.2 (Pin_2), J3.1 (Pin_1), J3.18 (Pin_18), J3.19 (Pin_19), J3.2 (Pin_2), J3.20 (Pin_20), J3.6 (Pin_6), R1.2, SW1.1, TP1.1, U1.1, U1.10, U1.13, U1.4, U1.7 (GND)
- net E: now reaches U3.10 (GPIO17/U1TXD/ADC2_CH6)
- net E: now also J3.10 (Pin_10)
- net A: now reaches U3.11 (GPIO18/U1RXD/ADC2_CH7/CLK_OUT3)
- net A: now also J3.11 (Pin_11)
- net B: now reaches U3.12 (GPIO8/TOUCH8/ADC1_CH7/SUBSPICS1)
- net B: now also J3.12 (Pin_12)
- net D-: now reaches U3.13 (GPIO19/U1RTS/ADC2_CH8/CLK_OUT2/USB_D-)
- net D-: now also J1.A7 (D-), J1.B7 (D-)
- net D+: now reaches U3.14 (GPIO20/U1CTS/ADC2_CH9/CLK_OUT1/USB_D+)
- net D+: now also J1.A6 (D+), J1.B6 (D+)
- net C: now reaches U3.15 (GPIO3/TOUCH3/ADC1_CH2)
- net C: now also J3.13 (Pin_13)
- net D: now reaches U3.17 (GPIO9/TOUCH9/ADC1_CH8/FSPIHD/SUBSPIHD)
- net D: now also J3.14 (Pin_14)
- net SCK: now reaches U3.18 (GPIO10/TOUCH10/ADC1_CH9/FSPICS0/FSPIIO4/SUBSPICS0)
- net SCK: now also U1.11
- net MOSI: now reaches U3.19 (GPIO11/TOUCH11/ADC2_CH0/FSPID/FSPIIO5/SUBSPID)
- net MOSI: now also U1.8
- net +3.3V: now reaches U3.2 (3V3)
- net +3.3V: now also U2.2 (VO), C1.1, C3.1, C4.1, C5.1, C7.1, Card1.4 (VDD), R2.2, U1.14 (VCC)
- net CS: now reaches U3.20 (GPIO12/TOUCH12/ADC2_CH1/FSPICLK/FSPIIO6/SUBSPICLK)
- net CS: now also U1.6
- net MISO: now reaches U3.21 (GPIO13/TOUCH13/ADC2_CH2/FSPIQ/FSPIIO7/SUBSPIQ)
- net MISO: now also U1.3
- net CLK: now reaches U3.22 (GPIO14/TOUCH14/ADC2_CH3/FSPIWP/FSPIDQS/SUBSPIWP)
- net CLK: now also J3.15 (Pin_15)
- net LAT: now reaches U3.23 (GPIO21)
- net LAT: now also J3.16 (Pin_16)
- net OE: now reaches U3.24 (GPIO47/SPICLK_P/SUBSPICLK_P_DIFF)
- net OE: now also J3.17 (Pin_17)
- net CD: now reaches U3.25 (GPIO48/SPICLK_N/SUBSPICLK_N_DIFF)
- net CD: now also Card1.9 (CD)
- net at U3.27 (GPIO0/BOOT): now also TP1.2
- net at U3.3 (EN): now also R3.2
- net R1: now reaches U3.4 (GPIO4/TOUCH4/ADC1_CH3)
- net R1: now also J3.3 (Pin_3)
- net G1: now reaches U3.5 (GPIO5/TOUCH5/ADC1_CH4)
- net G1: now also J3.4 (Pin_4)
- net B1: now reaches U3.6 (GPIO6/TOUCH6/ADC1_CH5)
- net B1: now also J3.5 (Pin_5)
- net R2: now reaches U3.7 (GPIO7/TOUCH7/ADC1_CH6)
- net R2: now also J3.7 (Pin_7)
- net G2: now reaches U3.8 (GPIO15/U0RTS/ADC2_CH4/XTAL_32K_P)
- net G2: now also J3.8 (Pin_8)
- net B2: now reaches U3.9 (GPIO16/U0CTS/ADC2_CH5/XTAL_32K_NH5)
- net B2: now also J3.9 (Pin_9)
- net at J1.A4 (VBUS), J1.A9 (VBUS), J1.B4 (VBUS)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: now also D1.2 (A)
- net at J1.A5 (CC1): now also J1.B5 (CC2), R1.1
- net +5V: now reaches U2.3 (VI)
- net +5V: now also C2.1, D1.1 (K), D3.1 (K)
- new net: D3.2 (A), J2.1 (Pin_1)
- new net: R5.2, U1.2
- new net: Card1.7 (DAT0(D0)), R4.1
- new net: R4.2, U1.9
- new net: C6.2, R3.1, SW1.2
- new net: R7.2, U1.12
- new net: Card1.2 (CDDAT3(CS)), R5.1
- new net: Card1.3 (CMD(DI)), R6.1
- new net: Card1.5 (CLK(SCLK)), R7.1
- new net: D2.2 (A), R2.1
- new net: R6.2, U1.5
- no-connect marks 0 -> 18
Other:
- moved on the sheet: J1, U2, U3
