File: CameraPosition/WS2812.kicad_sch (KiCad schematic)
At the start: 20 parts

Commit message: update
Parts:
- renumbered D3 to D10, D6 to D11, D9 to D12, D12 to D13, D15 to D14, D17 to D15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

Commit message: update
Connections:
- no-connect marks 0 -> 1
