File: CameraPosition/CameraPosition.kicad_pcb (KiCad board)
At the start: 2 copper layers, 60 x 60 mm, 39 parts, among them J1 USB_C_Receptacle_USB2.0, J2 Conn_01x24, Q1 Q_PMOS_GSD, SW1 SW_Push, SW2 SW_Push, U1 IP5306, U2 ESP32-S3-WROOM-1, U3 AMS1117, U4 GC9A01_IPS_display_SPI, U5 XC6206P122MR, U6 XC6206P282MR

Commit message: update
Parts:
- added D10: WS2812B, LED_SMD:LED_WS2812B_PLCC4_5.0x5.0mm_P3.2mm, B.Cu at (72.2, 50.2)
- added D11: WS2812B, LED_SMD:LED_WS2812B_PLCC4_5.0x5.0mm_P3.2mm, B.Cu at (97.5, 50.2)
- added D12: WS2812B, LED_SMD:LED_WS2812B_PLCC4_5.0x5.0mm_P3.2mm, B.Cu at (80.7, 43.6)
- added D13: WS2812B, LED_SMD:LED_WS2812B_PLCC4_5.0x5.0mm_P3.2mm, B.Cu at (72.2, 43.6)
- added D14: WS2812B, LED_SMD:LED_WS2812B_PLCC4_5.0x5.0mm_P3.2mm, B.Cu at (89.1, 50.2)
- added D15: WS2812B, LED_SMD:LED_WS2812B_PLCC4_5.0x5.0mm_P3.2mm, B.Cu at (105.9, 43.6)
- added D16: WS2812B, LED_SMD:LED_WS2812B_PLCC4_5.0x5.0mm_P3.2mm, B.Cu at (105.9, 50.2)
- added D17: WS2812B, LED_SMD:LED_WS2812B_PLCC4_5.0x5.0mm_P3.2mm, B.Cu at (80.7, 37.0)
- added D18: WS2812B, LED_SMD:LED_WS2812B_PLCC4_5.0x5.0mm_P3.2mm, B.Cu at (97.5, 37.0)
- added D19: WS2812B, LED_SMD:LED_WS2812B_PLCC4_5.0x5.0mm_P3.2mm, B.Cu at (80.7, 50.2)
- added D2: WS2812B, LED_SMD:LED_WS2812B_PLCC4_5.0x5.0mm_P3.2mm, B.Cu at (72.2, 37.0)
- added D20: WS2812B, LED_SMD:LED_WS2812B_PLCC4_5.0x5.0mm_P3.2mm, B.Cu at (97.5, 56.9)
- added D21: WS2812B, LED_SMD:LED_WS2812B_PLCC4_5.0x5.0mm_P3.2mm, B.Cu at (106.8, 61.9)
- added D3: WS2812B, LED_SMD:LED_WS2812B_PLCC4_5.0x5.0mm_P3.2mm, B.Cu at (89.1, 37.0)
- added D4: WS2812B, LED_SMD:LED_WS2812B_PLCC4_5.0x5.0mm_P3.2mm, B.Cu at (105.9, 37.0)
- added D5: WS2812B, LED_SMD:LED_WS2812B_PLCC4_5.0x5.0mm_P3.2mm, B.Cu at (97.5, 43.6)
- added D6: WS2812B, LED_SMD:LED_WS2812B_PLCC4_5.0x5.0mm_P3.2mm, B.Cu at (63.8, 37.0)
- added D7: WS2812B, LED_SMD:LED_WS2812B_PLCC4_5.0x5.0mm_P3.2mm, B.Cu at (80.7, 56.9)
- added D8: WS2812B, LED_SMD:LED_WS2812B_PLCC4_5.0x5.0mm_P3.2mm, B.Cu at (89.1, 43.6)
- added D9: WS2812B, LED_SMD:LED_WS2812B_PLCC4_5.0x5.0mm_P3.2mm, B.Cu at (89.1, 56.9)
- moved D2 18.7 mm to (100.0, 73.0)

Commit message: update
Parts:
- removed the D2 at (100.0, 73.0)
- removed the D2 at (72.2, 37.0)
- added D2: WS2812B, LED_SMD:LED_WS2812B_PLCC4_5.0x5.0mm_P3.2mm, B.Cu at (23.5, 57.3)
- moved J1 117.0 mm to (23.1, 49.0), turned to -90 degrees
- moved D21 85.6 mm to (22.2, 49.0), turned to 90 degrees
- moved J2 84.8 mm to (48.8, 30.6)
- moved U5 81.9 mm to (49.0, 58.8)
- moved D4 80.1 mm to (33.2, 70.7), turned to 144 degrees
- moved D20 75.7 mm to (23.5, 40.7), turned to 72 degrees
- moved D3 67.7 mm to (27.3, 64.8), turned to 126 degrees
- moved D18 65.0 mm to (33.2, 27.3), turned to 36 degrees
- moved D5 64.6 mm to (40.7, 74.5), turned to 162 degrees
- moved D16 63.5 mm to (49.0, 22.2), turned to 0 degrees
- moved D1 60.0 mm to (106.6, 59.6)
- moved U6 57.5 mm to (66.6, 49.5)
- moved D19 56.0 mm to (27.3, 33.2), turned to 54 degrees
- moved D15 52.6 mm to (57.3, 23.5), turned to -18 degrees
- moved D17 42.2 mm to (40.7, 23.5), turned to 18 degrees
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- renumbered C9 to C1, C13 to C10, C15 to C11, C3 to C12, C1 to C13, C2 to C14, C4 to C15, C10 to C2, C12 to C3, C14 to C4, C11 to C5, C8 to C6, C5 to C7, C6 to C8, C7 to C9, R7 to R1, R3 to R2, R2 to R3, R6 to R4, R4 to R5, R5 to R6, R1 to R7, SW2 to SW1, SW1 to SW2, TP2 to TP1, TP1 to TP2, U3 to U1, U5 to U2, U1 to U3, U6 to U4, U4 to U5, U2 to U6
Connections:
- D11 pad 4: Net-(D11-Pad4) -> Net-(D10-Pad2)
- D12 pad 4: Net-(D12-Pad4) -> Net-(D11-Pad2)
- D13 pad 2: unconnected-(D13-Pad2) -> Net-(D13-Pad2)
- D13 pad 4: Net-(D10-Pad2) -> Net-(D12-Pad2)
- D14 pad 4: Net-(D11-Pad2) -> Net-(D13-Pad2)
- D15 pad 4: Net-(D12-Pad2) -> Net-(D14-Pad2)
- D16 pad 4: Net-(D14-Pad2) -> Net-(D15-Pad2)
- D17 pad 4: Net-(D15-Pad2) -> Net-(D16-Pad2)
- D18 pad 4: Net-(D16-Pad2) -> Net-(D17-Pad2)
- D19 pad 4: Net-(D17-Pad2) -> Net-(D18-Pad2)
- D20 pad 4: Net-(D18-Pad2) -> Net-(D19-Pad2)
- D21 pad 2: Net-(D21-Pad2) -> unconnected-(D21-Pad2)
- D21 pad 4: Net-(D19-Pad2) -> Net-(D20-Pad2)
- D3 pad 4: Net-(D20-Pad2) -> Net-(D2-Pad2)
- D4 pad 4: Net-(D21-Pad2) -> Net-(D3-Pad2)
- D5 pad 4: Net-(D2-Pad2) -> Net-(D4-Pad2)
- D6 pad 4: Net-(D3-Pad2) -> Net-(D5-Pad2)
- D7 pad 2: Net-(D10-Pad4) -> Net-(D7-Pad2)
- D7 pad 4: Net-(D4-Pad2) -> Net-(D6-Pad2)
- D8 pad 2: Net-(D11-Pad4) -> Net-(D8-Pad2)
- D8 pad 4: Net-(D5-Pad2) -> Net-(D7-Pad2)
- D9 pad 2: Net-(D12-Pad4) -> Net-(D10-Pad4)
- D9 pad 4: Net-(D6-Pad2) -> Net-(D8-Pad2)
Other:
- outline, holes or cut-outs redrawn

Commit message: update
Parts:
- added C16: 0.1u, Capacitor_SMD:C_0805_2012Metric, F.Cu at (48.5, 56.0)
- added C17: 0.1u, Capacitor_SMD:C_0805_2012Metric, F.Cu at (48.0, 25.8)
- added C18: 1u, Capacitor_SMD:C_0805_2012Metric, B.Cu at (66.0, 35.5)
- added C19: 0.1u, Capacitor_SMD:C_0805_2012Metric, F.Cu at (61.0, 32.0)
- added C20: 10u, Capacitor_SMD:C_0805_2012Metric, F.Cu at (70.5, 31.5)
- added C21: 1u, Capacitor_SMD:C_0805_2012Metric, F.Cu at (72.0, 33.5)
- added C22: 0.1u, Capacitor_SMD:C_0805_2012Metric, F.Cu at (73.0, 35.5)
- added Q2: 2N7002, Package_TO_SOT_SMD:SOT-23, F.Cu at (36.0, 56.0)
- added Q3: 2N7002, Package_TO_SOT_SMD:SOT-23, F.Cu at (66.5, 59.2)
- added R10: 10k, Resistor_SMD:R_0805_2012Metric, F.Cu at (39.0, 56.0)
- added R11: 1K, Resistor_SMD:R_0805_2012Metric, F.Cu at (69.5, 35.5)
- added R12: 1K, Resistor_SMD:R_0805_2012Metric, F.Cu at (51.2, 25.8)
- added R13: 10k, Resistor_SMD:R_0805_2012Metric, F.Cu at (63.5, 59.2)
- added R8: 22, Resistor_SMD:R_0805_2012Metric, F.Cu at (40.0, 59.0)
- added R9: 10K, Resistor_SMD:R_0805_2012Metric, F.Cu at (53.2, 53.8)
- added TP3: TestPoint_2Pole, Connector_PinHeader_2.00mm:PinHeader_1x02_P2.00mm_Vertical, F.Cu at (66.0, 62.5)
- C1, C2: value 1u -> 10u
- C10: value 0.1u -> 10u
- C11, C8: value 10u -> 22u
- C12: value 1u -> 0.1u
- C14: value 1u -> 15p
- C3: value 0.1u -> 1u
- C4: value 10u -> 1u
- C5: value 10u -> 0.1u
- C6, C9: value 22u -> 10u
- D1, R3, SW1, SW2: moved to B.Cu
- J2: value Conn_01x24 -> Conn_01x25
- R7: value 1K -> 10k
- U3: footprint Package_SO:SOIC-8-1EP_3.9x4.9mm_P1.27mm_EP2.29x3mm_ThermalVias -> Package_SO:SOIC-8-1EP_3.9x4.9mm_P1.27mm_EP2.29x3mm
- moved R3 144.8 mm to (27.0, 46.7), turned to 90 degrees
- moved R1 139.8 mm to (31.5, 28.0), turned to -90 degrees
- moved C4 139.4 mm to (27.0, 35.0), turned to 90 degrees
- moved C7 133.2 mm to (35.0, 25.0)
- moved C3 128.9 mm to (33.0, 40.0)
- moved C10 126.9 mm to (31.6, 48.0), turned to 90 degrees
- moved R5 124.0 mm to (31.6, 51.5), turned to -90 degrees
- moved R6 122.6 mm to (35.0, 53.0)
- moved C12 122.5 mm to (55.2, 25.8), turned to -90 degrees
- moved Q1 122.4 mm to (34.5, 28.0)
- moved C9 121.8 mm to (29.6, 51.5), turned to 90 degrees
- moved R2 121.1 mm to (29.6, 48.0), turned to 90 degrees
- moved U2 119.1 mm to (56.0, 22.3)
- moved C2 117.8 mm to (38.5, 45.0)
- moved C13 117.6 mm to (53.2, 25.8), turned to -90 degrees
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Connections:
- BT1 pad 1: +3V8 -> /BAT
- C10 pad 2: +2V8 -> VCC
- C11 pad 2: +2V8 -> Net-(C11-Pad2)
- C12 pad 2: Net-(C12-Pad2) -> +2V8
- C13 pad 1: +3.3V -> GND
- C13 pad 2: GND -> +2V8
- C14 pad 1: +3.3V -> /CAM_PCLK
- C15 pad 1: +3.3V -> GND
- C15 pad 2: GND -> Net-(C15-Pad2)
- C2 pad 2: +3V3 -> +5V
- C3 pad 2: +1V2 -> +5V
- C4 pad 2: +1V2 -> +3V3
- C5 pad 2: Net-(C5-Pad2) -> +1V2
- C6 pad 2: +3V8 -> +1V2
- C8 pad 2: VCC -> /BAT
- D2 pad 4: /WS2812/DIN -> /LED_IN
- J1 pad A4: +5V -> VCC
- J1 pad A9: +5V -> VCC
- J1 pad B4: +5V -> VCC
- J1 pad B9: +5V -> VCC
- J2 pad 10: unconnected-(J2-Pad10) -> GND
- J2 pad 11: unconnected-(J2-Pad11) -> /CAM_D8
- J2 pad 12: unconnected-(J2-Pad12) -> /CAM_MCLK
- J2 pad 13: unconnected-(J2-Pad13) -> /CAM_D9
- J2 pad 14: unconnected-(J2-Pad14) -> +3V3
- J2 pad 15: unconnected-(J2-Pad15) -> +1V2
- J2 pad 16: unconnected-(J2-Pad16) -> /CAM_HSYNC
- J2 pad 17: unconnected-(J2-Pad17) -> Net-(J2-Pad17)
- J2 pad 18: unconnected-(J2-Pad18) -> /CAM_VSYNC
- J2 pad 19: unconnected-(J2-Pad19) -> /CAM_RST
- J2 pad 20: unconnected-(J2-Pad20) -> /CAM_SCK
- J2 pad 21: unconnected-(J2-Pad21) -> +2V8
- J2 pad 22: unconnected-(J2-Pad22) -> /CAM_SDA
- J2 pad 23: unconnected-(J2-Pad23) -> GND
- J2 pad 3: unconnected-(J2-Pad3) -> /CAM_D4
- J2 pad 4: unconnected-(J2-Pad4) -> /CAM_D3
- J2 pad 5: unconnected-(J2-Pad5) -> /CAM_D5
- J2 pad 6: unconnected-(J2-Pad6) -> /CAM_D2
- J2 pad 7: unconnected-(J2-Pad7) -> /CAM_D6
- J2 pad 8: unconnected-(J2-Pad8) -> /CAM_PCLK
- J2 pad 9: unconnected-(J2-Pad9) -> /CAM_D7
- L1 pad 2: +3V8 -> /BAT
- Q1 pad 3: Net-(C5-Pad2) -> Net-(C7-Pad2)
- R2 pad 1: Net-(C7-Pad2) -> Net-(C9-Pad2)
- R4 pad 1: Net-(C9-Pad2) -> Net-(C11-Pad2)
- R4 pad 2: +3V8 -> /BAT
- R7 pad 1: Net-(C12-Pad2) -> +3V3
- R7 pad 2: Net-(R7-Pad2) -> /CAM_RST
- SW2 pad 2: Net-(C12-Pad2) -> Net-(C18-Pad2)
- U2 pad 3: Net-(C5-Pad2) -> Net-(C7-Pad2)
- U3 pad 3: +3V8 -> /BAT
- U3 pad 4: +3V8 -> /BAT
- U3 pad 6: Net-(C9-Pad2) -> Net-(C11-Pad2)
- U4 pad 3: Net-(C5-Pad2) -> Net-(C7-Pad2)
- U5 pad 1: unconnected-(U5-Pad1) -> GND
- U5 pad 10: unconnected-(U5-Pad10) -> /DIS_SDI
- U5 pad 11: unconnected-(U5-Pad11) -> Net-(C15-Pad2)
- U5 pad 12: unconnected-(U5-Pad12) -> GND
- U5 pad 2: unconnected-(U5-Pad2) -> Net-(R8-Pad2)
- U5 pad 3: unconnected-(U5-Pad3) -> +3V3
- U5 pad 4: unconnected-(U5-Pad4) -> +3V3
- U5 pad 5: unconnected-(U5-Pad5) -> GND
- U5 pad 6: unconnected-(U5-Pad6) -> GND
- U5 pad 7: unconnected-(U5-Pad7) -> /DIS_DC
- U5 pad 8: unconnected-(U5-Pad8) -> GND
- U5 pad 9: unconnected-(U5-Pad9) -> /DIS_SCK
- U6 pad 10: unconnected-(U6-Pad10) -> /CAM_D8
- U6 pad 11: unconnected-(U6-Pad11) -> /CAM_D7
- U6 pad 12: unconnected-(U6-Pad12) -> /CAM_PCLK
- U6 pad 15: unconnected-(U6-Pad15) -> /CAM_D6
- U6 pad 17: unconnected-(U6-Pad17) -> /CAM_D2
- U6 pad 18: unconnected-(U6-Pad18) -> /CAM_D5
- U6 pad 19: unconnected-(U6-Pad19) -> /CAM_D3
- U6 pad 2: +3.3V -> +3V3
- U6 pad 20: unconnected-(U6-Pad20) -> /CAM_D4
- U6 pad 21: unconnected-(U6-Pad21) -> /DIS_DC
- U6 pad 22: unconnected-(U6-Pad22) -> /DIS_SCK
- U6 pad 23: unconnected-(U6-Pad23) -> /DIS_SDI
- U6 pad 24: unconnected-(U6-Pad24) -> /LED_IN
- U6 pad 3: Net-(R7-Pad2) -> Net-(R11-Pad2)
- U6 pad 4: unconnected-(U6-Pad4) -> /CAM_SDA
- U6 pad 5: unconnected-(U6-Pad5) -> /CAM_SCK
- U6 pad 6: unconnected-(U6-Pad6) -> /CAM_VSYNC
- U6 pad 7: unconnected-(U6-Pad7) -> /CAM_HSYNC
- U6 pad 8: unconnected-(U6-Pad8) -> /CAM_D9
- U6 pad 9: unconnected-(U6-Pad9) -> /CAM_MCLK
Routing:
- net /D-: track 0.00 -> 46.5 mm, vias 0 -> 2
- net /D+: track 0.00 -> 40.7 mm, vias 0 -> 2
- net +3V3: track 0.00 -> 37.3 mm, vias 0 -> 12
- net /LED_IN: track 0.00 -> 33.2 mm, vias 0 -> 1
- net Net-(C7-Pad2): track 0.00 -> 31.2 mm, vias 0 -> 2
- net /CAM_D4: track 0.00 -> 22.3 mm
- net /CAM_SDA: track 0.00 -> 22.0 mm
- net /CAM_VSYNC: track 0.00 -> 21.2 mm
- net /CAM_HSYNC: track 0.00 -> 21.1 mm
- net /CAM_D3: track 0.00 -> 20.8 mm
- net /CAM_SCK: track 0.00 -> 20.8 mm
- net /CAM_D9: track 0.00 -> 20.5 mm
- net /CAM_PCLK: track 0.00 -> 20.3 mm
- net /CAM_MCLK: track 0.00 -> 20.1 mm
- net /CAM_D8: track 0.00 -> 19.5 mm
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- added copper zone on In1.Cu, net +3V3
- added copper zone on B.Cu, net +5V
- added copper zone on F.Cu, net GND
- added copper zone on In2.Cu, net GND
Other:
- outline, holes or cut-outs redrawn
- copper layers 2 -> 4

Commit message: update
Parts:
- added G***: LOGO, 1Use:Hockey, B.Cu at (33.7, 33.8)
Other:
- board size 60 x 60 mm -> 62 x 62 mm
- board text added: "+"
- board text added: "-"
- board text added: "By Andy 230305"
