File: CameraPosition/CameraPosition.kicad_sch (KiCad schematic)
At the start: 2 parts

Commit message: update
Parts:
- J?: footprint (none) -> 1Use:USB_C_Receptacle_HRO_TYPE-C-31-M-12
Changed lines of the file:
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@@
     (property "Reference" "J?" (id 0) (at 35.56 19.05 0))
     (property "Value" "USB_C_Receptacle_USB2.0" (id 1) (at 35.56 21.59 0))
-    (property "Footprint" "" (id 2) (at 39.37 41.91 0)
+    (property "Footprint" "1Use:USB_C_Receptacle_HRO_TYPE-C-31-M-12" (id 2) (at 39.37 41.91 0)
       (effects (font (size 1.27 1.27)) hide)
     )
@@
   (symbol_instances
     (path "/50a07654-ad9a-4b65-8721-d7fba80ecbea"
-      (reference "J?") (unit 1) (value "USB_C_Receptacle_USB2.0") (footprint "")
+      (reference "J?") (unit 1) (value "USB_C_Receptacle_USB2.0") (footprint "1Use:USB_C_Receptacle_HRO_TYPE-C-31-M-12")
     )
     (path "/214a9b78-19cc-43c0-9584-e9945c2cdbc4"

Commit message: update
Parts:
- added BT?: Battery_Cell, Connector_PinHeader_2.54mm:PinHeader_1x02_P2.54mm_Vertical, symbol Device:Battery_Cell
- added C? (x2): 1u, Capacitor_SMD:C_0805_2012Metric, symbol 1CommonUse:C0805
- added C? (x5): 10u, Capacitor_SMD:C_0805_2012Metric, symbol 0805:C
- added C? (x2): 22u, Capacitor_SMD:C_0805_2012Metric, symbol 0805:C
- added C? (x2): 0.1u, Capacitor_SMD:C_0805_2012Metric, symbol 0805:C
- added C? (x2): 1u, Capacitor_SMD:C_0805_2012Metric, symbol 0805:C
- added C?: 0.1u, Capacitor_SMD:C_0805_2012Metric, symbol 1CommonUse:C0805
- added C?: 10u, Capacitor_SMD:C_0805_2012Metric, symbol 1CommonUse:C0805
- added D?: LED, LED_SMD:LED_0805_2012Metric, symbol 0805:LED
- added D?: WS2812B, LED_SMD:LED_WS2812B_PLCC4_5.0x5.0mm_P3.2mm, symbol LED:WS2812B
- added J?: Conn_01x24, symbol Connector_Generic:Conn_01x24
- added L?: 1n, Inductor_SMD:L_Wuerth_MAPI-2512, symbol Device:L_Small
- added Q?: Q_PMOS_GSD, Package_TO_SOT_SMD:SOT-23, symbol Device:Q_PMOS_GSD
- added R?: 0.5, Resistor_SMD:R_0805_2012Metric, symbol 0805:R
- added R? (x2): 10k, Resistor_SMD:R_0805_2012Metric, symbol 0805:R
- added R?: 2, Resistor_SMD:R_0805_2012Metric, symbol 0805:R
- added R?: 1K, Resistor_SMD:R_0805_2012Metric, symbol 1CommonUse:R0805
- added R?: 5.1K, Resistor_SMD:R_0805_2012Metric, symbol 1CommonUse:R0805
- added R?: 1K, Resistor_SMD:R_0805_2012Metric, symbol 0805:R
- added SW?: SW_Push, Button_Switch_SMD:SW_SPST_CK_RS282G05A3, symbol Switch:SW_Push
- added SW?: SW_Push, Button_Switch_SMD:SW_SPST_CK_RS282G05A3, symbol Resource:SW_Push
- added TP? (x2): TestPoint_2Pole, Connector_PinHeader_2.00mm:PinHeader_1x02_P2.00mm_Vertical, symbol Connector:TestPoint_2Pole
- added U?: XC6206P122MR, Package_TO_SOT_SMD:SOT-23, symbol Regulator_Linear:XC6206PxxxMR
- added U?: XC6206P282MR, Package_TO_SOT_SMD:SOT-23, symbol Regulator_Linear:XC6206PxxxMR
- added U?: AMS1117, Package_TO_SOT_SMD:SOT-223-3_TabPin2, symbol Regulator_Linear:AMS1117
- added U?: IP5306, Package_SO:SOIC-8-1EP_3.9x4.9mm_P1.27mm_EP2.29x3mm_ThermalVias, symbol Resource:IP5306
Connections:
- net GND: now reaches U?.1 (GND)
- net GND: now also J?.A1 (GND), J?.A12 (GND), J?.B1 (GND), J?.B12 (GND), J?.S1 (SHIELD), U?.40 (GND), U?.41 (GND), BT?.2 (-), C?.1, C?.1, C?.1, C?.1, C?.1, C?.1, C?.1, C?.1, C?.1, C?.1, C?.1, C?.1, C?.2, C?.2, C?.2, D?.1 (K), R?.2, SW?.1, SW?.2, TP?.1, TP?.1, U?.1 (ADJ), U?.1 (GND), U?.1 (GND), U?.9 (GND)
- net D-: now reaches U?.13 (GPIO19/U1RTS/ADC2_CH8/CLK_OUT2/USB_D-)
- net D-: now also J?.A7 (D-), J?.B7 (D-)
- net D+: now reaches U?.14 (GPIO20/U1CTS/ADC2_CH9/CLK_OUT1/USB_D+)
- net D+: now also J?.A6 (D+), J?.B6 (D+)
- net +3.3V: now reaches U?.2 (3V3)
- net +3.3V: now also C?.1, C?.1, C?.1
- net at U?.27 (GPIO0/BOOT): now also TP?.2
- net at U?.3 (EN): now also R?.2
- net +5V: now reaches J?.A4 (VBUS), J?.A9 (VBUS), J?.B4 (VBUS), J?.B9 (VBUS)
- net +5V: now also C?.2, U?.3 (VI), U?.8 (VOUT)
- net at J?.A5 (CC1): now also J?.B5 (CC2), R?.1
- new net: C?.2, Q?.3 (D), U?.3 (VI), U?.3 (VI)
- new net: C?.2, R?.1, U?.6 (BAT)
- new net: C?.2, R?.1
- new net: L?.1, U?.7 (SW)
- new net: C?.2, R?.1, SW?.2
- new net: D?.2 (A), R?.1
- new net: R?.2, U?.2 (LED1)
- new net: R?.2, U?.5 (KEY)
- new net +1V2: C?.2, C?.2, U?.2 (VO)
- new net +2V8: C?.2, C?.2, U?.2 (VO)
- new net +3V3: C?.2, Q?.2 (S), R?.2, U?.2 (VO)
- new net +3V8: BT?.1 (+), C?.2, L?.2, R?.2, U?.3 (LED2), U?.4 (LED3)
- new net CAM_PWR: Q?.1 (G), R?.1
- new net D13: R?.1, SW?.1, TP?.2
- new net VCC: C?.2, R?.2, U?.1 (VIN)
- no-connect marks 0 -> 2
Other:
- moved on the sheet: U?

Commit message: update
Parts:
- added U4: GC9A01_IPS_display_SPI, 1Use:GC9A01_IPS_display, symbol gc9a01_ips_display_spi:GC9A01_IPS_display_SPI
- J2: renamed from J?; footprint (none) -> 1Use:Hirose_FH12-24S-0.5SH_1x24-1MP_P0.50mm_Horizontal
- gave numbers to parts that had none: 37

Commit message: update
Parts:
- removed D2: WS2812B, LED_SMD:LED_WS2812B_PLCC4_5.0x5.0mm_P3.2mm, symbol LED:WS2812B
Other:
- added sheet WS2812 (WS2812.kicad_sch)
- moved on the sheet: J2

Commit message: update
Parts:
- renumbered C9 to C1, C13 to C10, C15 to C11, C3 to C12, C1 to C13, C2 to C14, C4 to C15, C10 to C2, C12 to C3, C14 to C4, C11 to C5, C8 to C6, C5 to C7, C6 to C8, C7 to C9, R7 to R1, R3 to R2, R2 to R3, R6 to R4, R4 to R5, R5 to R6, R1 to R7, SW2 to SW1, SW1 to SW2, TP2 to TP1, TP1 to TP2, U3 to U1, U5 to U2, U1 to U3, U6 to U4, U4 to U5, U2 to U6

Commit message: update
Parts:
- removed J2: Conn_01x24, 1Use:Hirose_FH12-24S-0.5SH_1x24-1MP_P0.50mm_Horizontal, symbol Connector_Generic:Conn_01x24
- removed SW1: SW_Push, Button_Switch_SMD:SW_SPST_CK_RS282G05A3, symbol Resource:SW_Push
- removed U3: IP5306, Package_SO:SOIC-8-1EP_3.9x4.9mm_P1.27mm_EP2.29x3mm_ThermalVias, symbol Resource:IP5306
- added C1, C2: 10u, Capacitor_SMD:C_0805_2012Metric, symbol 0805:C
- added C14: 15p, Capacitor_SMD:C_0805_2012Metric, symbol 0805:C
- added C15, C16, C17, C19: 0.1u, Capacitor_SMD:C_0805_2012Metric, symbol 0805:C
- added J2: Conn_01x25, 1Use:Hirose_FH12-24S-0.5SH_1x24-1MP_P0.50mm_Horizontal, symbol Connector_Generic:Conn_01x25
- added Q2, Q3: 2N7002, Package_TO_SOT_SMD:SOT-23, symbol Transistor_FET:2N7002
- added R10, R13, R7: 10k, Resistor_SMD:R_0805_2012Metric, symbol 0805:R
- added R12: 1K, Resistor_SMD:R_0805_2012Metric, symbol 0805:R
- added R8: 22, Resistor_SMD:R_0805_2012Metric, symbol 0805:R
- added R9: 10K, Resistor_SMD:R_0805_2012Metric, symbol 0805:R
- added SW1: SW_Push, Button_Switch_SMD:SW_SPST_CK_RS282G05A3, symbol Switch:SW_Push
- added TP3: TestPoint_2Pole, Connector_PinHeader_2.00mm:PinHeader_1x02_P2.00mm_Vertical, symbol Connector:TestPoint_2Pole
- added U3: IP5306, Package_SO:SOIC-8-1EP_3.9x4.9mm_P1.27mm_EP2.29x3mm, symbol ip5306:IP5306
- renumbered C8 to C10, C9 to C11, C10 to C12, C11 to C13, C12 to C18, C13 to C20, C14 to C21, C15 to C22, C1 to C3, C2 to C4, C3 to C5, C4 to C6, C5 to C7, C6 to C8, C7 to C9, R7 to R11
Connections:
- net +3.3V is gone; now on net +3V3: C20.1, C21.1, C22.1, U6.2 (3V3)
- net +1V2: now also J2.15 (Pin_15)
- net +2V8: now also J2.21 (Pin_21)
- net +3V3: now also U5.3 (LEDA), U5.4 (VDD), C16.2, C17.1, J2.14 (Pin_14), R7.1, R9.2, TP3.2
- net +5V: now also C1.2, C2.2, U3.8 (VOUT); no longer J1.A4 (VBUS), J1.A9 (VBUS), J1.B4 (VBUS), J1.B9 (VBUS)
- net D13: now also SW1.1
- net GND: now also U5.1 (GND), U5.12 (GND), U5.5 (GND), U5.6 (GND), U5.8 (~{CS}), C1.1, C14.2, C15.1, C16.1, C17.2, C19.2, C2.1, J2.10 (Pin_10), J2.23 (Pin_23), J2.25 (Pin_25), Q2.2 (S), Q3.2 (S), R10.2, R12.1, R13.2, SW1.2, U3.9 (GND)
- net VCC: now also J1.A4 (VBUS), J1.A9 (VBUS), J1.B4 (VBUS), J1.B9 (VBUS), U3.1 (VIN)
- net CAM_D8: now reaches U6.10 (GPIO17/U1TXD/ADC2_CH6)
- net CAM_D8: now also J2.11 (Pin_11)
- net CAM_D7: now reaches U6.11 (GPIO18/U1RXD/ADC2_CH7/CLK_OUT3)
- net CAM_D7: now also J2.9 (Pin_9)
- net CAM_PCLK: now reaches U6.12 (GPIO8/TOUCH8/ADC1_CH7/SUBSPICS1)
- net CAM_PCLK: now also C14.1, J2.8 (Pin_8)
- net CAM_D6: now reaches U6.15 (GPIO3/TOUCH3/ADC1_CH2)
- net CAM_D6: now also J2.7 (Pin_7)
- net CAM_D2: now reaches U6.17 (GPIO9/TOUCH9/ADC1_CH8/FSPIHD/SUBSPIHD)
- net CAM_D2: now also J2.6 (Pin_6)
- net CAM_D5: now reaches U6.18 (GPIO10/TOUCH10/ADC1_CH9/FSPICS0/FSPIIO4/SUBSPICS0)
- net CAM_D5: now also J2.5 (Pin_5)
- net CAM_D3: now reaches U6.19 (GPIO11/TOUCH11/ADC2_CH0/FSPID/FSPIIO5/SUBSPID)
- net CAM_D3: now also J2.4 (Pin_4)
- net CAM_D4: now reaches U6.20 (GPIO12/TOUCH12/ADC2_CH1/FSPICLK/FSPIIO6/SUBSPICLK)
- net CAM_D4: now also J2.3 (Pin_3)
- net DIS_DC: now reaches U6.21 (GPIO13/TOUCH13/ADC2_CH2/FSPIQ/FSPIIO7/SUBSPIQ)
- net DIS_DC: now also U5.7 (D/C)
- net DIS_SCK: now reaches U6.22 (GPIO14/TOUCH14/ADC2_CH3/FSPIWP/FSPIDQS/SUBSPIWP)
- net DIS_SCK: now also U5.9 (SCK)
- net DIS_SDI: now reaches U6.23 (GPIO21)
- net DIS_SDI: now also U5.10 (SDI)
- net LED_IN: now reaches U6.24 (GPIO47/SPICLK_P/SUBSPICLK_P_DIFF)
- net CAM_SDA: now reaches U6.4 (GPIO4/TOUCH4/ADC1_CH3)
- net CAM_SDA: now also J2.22 (Pin_22)
- net CAM_SCK: now reaches U6.5 (GPIO5/TOUCH5/ADC1_CH4)
- net CAM_SCK: now also J2.20 (Pin_20)
- net CAM_VSYNC: now reaches U6.6 (GPIO6/TOUCH6/ADC1_CH5)
- net CAM_VSYNC: now also J2.18 (Pin_18)
- net CAM_HSYNC: now reaches U6.7 (GPIO7/TOUCH7/ADC1_CH6)
- net CAM_HSYNC: now also J2.16 (Pin_16)
- net CAM_D9: now reaches U6.8 (GPIO15/U0RTS/ADC2_CH4/XTAL_32K_P)
- net CAM_D9: now also J2.13 (Pin_13)
- net CAM_MCLK: now reaches U6.9 (GPIO16/U0CTS/ADC2_CH5/XTAL_32K_NH5)
- net CAM_MCLK: now also J2.12 (Pin_12)
- net at C11.2, R4.1: now also U3.6 (BAT)
- net at L1.1: now also U3.7 (SW)
- net at U5.11 (~{RESET}): now also C15.2, R9.1
- net at U5.2 (LEDK): now also R8.2
- net at R5.2: now also U3.2 (LED1)
- net at R6.2: now also U3.5 (KEY)
- net +3V8 renamed BAT
- net BAT: now also U3.3 (LED2), U3.4 (LED3)
- new net: J2.17 (Pin_17), R12.2
- new net: Q2.3 (D), R8.1
- new net: Q3.3 (D), TP3.1
- new net CAM_RST: C19.1, J2.19 (Pin_19), R7.2
- new net DIS_LED: Q2.1 (G), R10.1
- new net Motor: Q3.1 (G), R13.1
- no-connect marks 2 -> 20
Other:
- sheet WS2812 ports: added none; removed 5V, GND
- moved on the sheet: C18, C20, C21, C22, R11, SW2, TP2, U5, U6

Commit message: update
Parts:
- L1: value 1n -> 1u
Changed lines of the file:
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@@
     (in_bom yes) (on_board yes)
     (property "Reference" "L1" (id 0) (at 135.89 28.321 90))
-    (property "Value" "1n" (id 1) (at 135.89 30.6324 90))
+    (property "Value" "1u" (id 1) (at 135.89 30.6324 90))
     (property "Footprint" "Inductor_SMD:L_Wuerth_MAPI-2512" (id 2) (at 135.89 33.02 0)
       (effects (font (size 1.27 1.27)) hide)
@@
     )
     (path "/5a5b7060-983c-4989-878e-3126720e998d"
-      (reference "L1") (unit 1) (value "1n") (footprint "Inductor_SMD:L_Wuerth_MAPI-2512")
+      (reference "L1") (unit 1) (value "1u") (footprint "Inductor_SMD:L_Wuerth_MAPI-2512")
     )
     (path "/203bddf5-889d-4566-ba36-fe7a8bede16e"
